File: ozinverterkicad.sch (KiCad schematic (older format))
At the start: 68 parts, among them P1 CONN_02X05, P2 CONN_01X02, P3 on/off, P4 temp, P5 ct sense, P6 Active mains, P7 neutral mains, P8 systemled, Q1 tip35c, Q2 tip35c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

Commit message: reworked with connector changes
Parts:
- C23: footprint Capacitors_ThroughHole:C_Radial_D5_L6_P2.5 -> Capacitors_ThroughHole:C_Rect_L27_W11_P22
- D14, D5: symbol LED -> LED-RESCUE-ozinverterkicad
- RV1, voltageout1: symbol POT -> POT-RESCUE-ozinverterkicad
- Y1: footprint Crystals:Crystal_HC48-U_Vertical -> Crystals:Crystal_HC49-U_Vertical
Connections:
- net +48V: now also P1.1 (P1), P1.2 (P2); no longer P1.10 (P10), P1.9 (P9)
- net GND: now also P1.10 (P10), P1.9 (P9); no longer P1.1 (P1), P1.2 (P2)
- net at P1.3 (P3): now also U1.7 (ho); no longer U1.1 (LO)
- net at P1.7 (P7): now also U1.1 (LO); no longer U1.7 (ho)
Changed lines of the file:
@@
 EESchema Schematic File Version 2
+LIBS:ozinverterkicad-rescue
 LIBS:power
 LIBS:device
@@
 LIBS:valves
 LIBS:ozinverterlib
+LIBS:ozinverterkicad-cache
 EELAYER 25 0
 EELAYER END
@@
 $EndComp
 $Comp
-L LED D5
+L LED-RESCUE-ozinverterkicad D5
 U 1 1 57CA8B3C
 P 5725 4575
@@
 F 0 "Y1" H 6275 3650 50  0000 C CNN
 F 1 "12MHZ Crystal" H 6200 3700 50  0000 C CNN
-F 2 "Crystals:Crystal_HC48-U_Vertical" H 6275 3500 50  0001 C CNN
+F 2 "Crystals:Crystal_HC49-U_Vertical" H 6275 3500 50  0001 C CNN
 F 3 "" H 6275 3500 50  0000 C CNN
 	1    6275 3500
@@
 $EndComp
 $Comp
-L POT voltageout1
+L POT-RESCUE-ozinverterkicad voltageout1
 U 1 1 57CA98D3
 P 7450 4175
@@
 F 0 "C23" H 9250 3800 50  0000 L CNN
 F 1 "2uf" H 9250 3600 50  0000 L CNN
-F 2 "Capacitors_ThroughHole:C_Radial_D5_L6_P2.5" H 9263 3550 50  0001 C CNN
+F 2 "Capacitors_ThroughHole:C_Rect_L27_W11_P22" H 9263 3550 50  0001 C CNN
 F 3 "" H 9225 3700 50  0000 C CNN
 	1    9225 3700
@@
 $EndComp
 $Comp
-L POT RV1
+L POT-RESCUE-ozinverterkicad RV1
 U 1 1 57CAB4A0
 P 7000 2775
@@
 L GND #PWR019
 U 1 1 57CB3A5E
-P 1500 7400
-F 0 "#PWR019" H 1500 7150 50  0001 C CNN
-F 1 "GND" H 1500 7250 50  0000 C CNN
-F 2 "" H 1500 7400 50  0000 C CNN
-F 3 "" H 1500 7400 50  0000 C CNN
-	1    1500 7400
+P 1100 6475
+F 0 "#PWR019" H 1100 6225 50  0001 C CNN
+F 1 "GND" H 1100 6325 50  0000 C CNN
+F 2 "" H 1100 6475 50  0000 C CNN
+F 3 "" H 1100 6475 50  0000 C CNN
+	1    1100 6475
 	1    0    0    -1
 $EndComp
@@
 L +48V #PWR020
 U 1 1 57CB3D96
-P 1375 6550
-F 0 "#PWR020" H 1375 6400 50  0001 C CNN
-F 1 "+48V" H 1375 6690 50  0000 C CNN
-F 2 "" H 1375 6550 50  0000 C CNN
-F 3 "" H 1375 6550 50  0000 C CNN
-	1    1375 6550
+P 1775 7575
+F 0 "#PWR020" H 1775 7425 50  0001 C CNN
+F 1 "+48V" H 1775 7715 50  0000 C CNN
+F 2 "" H 1775 7575 50  0000 C CNN
+F 3 "" H 1775 7575 50  0000 C CNN
+	1    1775 7575
 	1    0    0    -1
 $EndComp
@@
 	4975 4550 4975 4625
 Wire Wire Line
-	5025 4075 5025 3975
+	5025 3975 5025 4075
 Wire Wire Line
 	5125 3975 5125 4075
@@
 	7425 3500 7425 3900
 Wire Wire Line
-	7100 3900 7100 3525
+	7100 3525 7100 3900
 Wire Wire Line
 	7100 3525 7175 3525
@@
 	6250 2650 6475 2650
 Wire Wire Line
-	5975 3175 6475 3175
-Wire Wire Line
-	6475 3175 6475 2950
+	6475 3175 5975 3175
+Wire Wire Line
+	6475 2950 6475 3175
 Wire Wire Line
 	6475 3050 6550 3050
@@
 	6000 1725 6000 1775
 Wire Wire Line
-	5975 3075 6150 3075
-Wire Wire Line
-	6150 3075 6150 1425
-Wire Wire Line
-	6150 1425 6000 1425
+	6150 3075 5975 3075
+Wire Wire Line
+	6150 1425 6150 3075
+Wire Wire Line
+	6000 1425 6150 1425
 Connection ~ 6075 1425
 Wire Wire Line
@@
 Connection ~ 2100 2925
 Wire Wire Line
-	1775 3075 1775 2850
+	1775 2850 1775 3075
 Wire Wire Line
 	1775 2850 2375 2850
@@
 	1675 6625 1675 6850
 Wire Wire Line
-	1375 6550 1375 6625
+	1375 6475 1375 6625
 Connection ~ 1375 6625
 Wire Wire Line
@@
 Connection ~ 2025 4475
 Wire Wire Line
-	1700 4625 1700 4400
+	1700 4400 1700 4625
 Wire Wire Line
 	1700 4400 2300 4400
@@
 	850  6300 1875 6300
 Wire Wire Line
-	1875 6300 1875 7150
-Wire Wire Line
-	1875 7150 1675 7150
+	1875 6300 1875 6950
 Wire Wire Line
 	1700 4600 950  4600
@@
 	1050 6150 1975 6150
 Wire Wire Line
-	1975 6150 1975 6950
-Wire Wire Line
-	1975 6950 1675 6950
+	1975 6150 1975 7150
 Wire Wire Line
 	4150 4175 4150 3475
@@
 	1500 1200 1500 1175
 Wire Wire Line
-	1375 1650 1375 1600
+	1375 1600 1375 1650
 Wire Wire Line
 	1150 950  1150 875
@@
 	3800 1225 3800 1200
 Wire Wire Line
-	3675 1675 3675 1625
+	3675 1575 3675 1675
 Wire Wire Line
 	3450 975  3450 900
@@
 Wire Wire Line
 	4450 1250 4425 1250
-Wire Wire Line
-	3675 1650 3675 1575
 Wire Wire Line
 	3675 1575 4300 1575
@@
 	4975 1200 4975 1025
 $Comp
-L LED D14
+L LED-RESCUE-ozinverterkicad D14
 U 1 1 57CC6041
 P 4725 1500
@@
 Wire Wire Line
 	5075 1350 5075 1025
+Wire Wire Line
+	1875 6950 1675 6950
+Connection ~ 1875 6950
+Wire Wire Line
+	1975 7150 1675 7150
+Wire Wire Line
+	1100 6475 1375 6475
+Connection ~ 1500 7400
+Wire Wire Line
+	1525 7400 1525 7575
+Wire Wire Line
+	1525 7575 1775 7575
+Connection ~ 1525 7400
 $EndSCHEMATC
